File: kicad/k1-aioc/k1-aioc.kicad_pcb (KiCad board)
At the start: 2 copper layers, 21 x 31.5 mm, 49 parts, among them J1 12401832E402A, J2 Conn_01x07_Male, Q1 BC847BS, U1 MIC5330-SSYML, U2 STM32F373CBTx, Y1 8MHz/20pF

Commit message: Changed naming of microcontroller IO pins to IN/OUT
Connections:
- net /PTT1 renamed /OUT1
- net /PTT1-IN renamed /IN1
- net /PTT2 renamed /OUT2
- net /PTT2-IN renamed /IN2
Changed lines of the file:
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@@
   (net 9 "unconnected-(U2-Pad40)")
   (net 10 "Net-(D1-Pad2)")
-  (net 11 "/PTT1-IN")
+  (net 11 "/OUT2")
   (net 12 "/SWCLK")
   (net 13 "unconnected-(U2-Pad15)")
@@
   (net 37 "Net-(Q1-Pad6)")
   (net 38 "/USART-TX")
-  (net 39 "/PTT1")
-  (net 40 "/PTT2")
+  (net 39 "/OUT1")
+  (net 40 "/IN2")
   (net 41 "/AFIN")
   (net 42 "/RADIO-MIC")
@@
   (net 58 "Net-(C5-Pad1)")
   (net 59 "/DAC_ATTEN")
-  (net 60 "/PTT2-IN")
+  (net 60 "/IN1")
   (net 61 "/RADIO-PTT1")
   (footprint "Resistor_SMD:R_0603_1608Metric" (layer "F.Cu")
@@
       (net 61 "/RADIO-PTT1") (pintype "passive"))
     (pad "2" smd roundrect (at 0.825 0 180) (size 0.8 0.95) (layers "F.Cu" "F.Paste" "F.Mask") (roundrect_rratio 0.25)
-      (net 11 "/PTT1-IN") (pintype "passive"))
+      (net 60 "/IN1") (pintype "passive"))
     (model "${KICAD6_3DMODEL_DIR}/Resistor_SMD.3dshapes/R_0603_1608Metric.wrl"
       (offset (xyz 0 0 0))
@@
       (net 47 "/RADIO-PTT2") (pintype "passive"))
     (pad "2" smd roundrect (at 0.825 0 180) (size 0.8 0.95) (layers "F.Cu" "F.Paste" "F.Mask") (roundrect_rratio 0.25)
-      (net 60 "/PTT2-IN") (pintype "passive"))
+      (net 40 "/IN2") (pintype "passive"))
     (model "${KICAD6_3DMODEL_DIR}/Resistor_SMD.3dshapes/R_0603_1608Metric.wrl"
       (offset (xyz 0 0 0))
@@
     (fp_line (start 0.8 0.4125) (end -0.8 0.4125) (layer "F.Fab") (width 0.1))
     (pad "1" smd roundrect (at -0.825 0 270) (size 0.8 0.95) (layers "F.Cu" "F.Paste" "F.Mask") (roundrect_rratio 0.25)
-      (net 39 "/PTT1") (pintype "passive"))
+      (net 39 "/OUT1") (pintype "passive"))
     (pad "2" smd roundrect (at 0.825 0 270) (size 0.8 0.95) (layers "F.Cu" "F.Paste" "F.Mask") (roundrect_rratio 0.25)
       (net 55 "Net-(Q1-Pad5)") (pintype "passive"))
@@
       (net 28 "+3.3VA") (pinfunction "VDDA") (pintype "power_in"))
     (pad "10" smd roundrect (at -4.1625 1.75 90) (size 1.475 0.3) (layers "F.Cu" "F.Paste" "F.Mask") (roundrect_rratio 0.25)
-      (net 40 "/PTT2") (pinfunction "PA0") (pintype "bidirectional"))
+      (net 11 "/OUT2") (pinfunction "PA0") (pintype "bidirectional"))
     (pad "11" smd roundrect (at -4.1625 2.25 90) (size 1.475 0.3) (layers "F.Cu" "F.Paste" "F.Mask") (roundrect_rratio 0.25)
-      (net 39 "/PTT1") (pinfunction "PA1") (pintype "bidirectional"))
+      (net 39 "/OUT1") (pinfunction "PA1") (pintype "bidirectional"))
     (pad "12" smd roundrect (at -4.1625 2.75 90) (size 1.475 0.3) (layers "F.Cu" "F.Paste" "F.Mask") (roundrect_rratio 0.25)
       (net 56 "unconnected-(U2-Pad12)") (pinfunction "PA2") (pintype "bidirectional"))
@@
       (net 26 "unconnected-(U2-Pad41)") (pinfunction "PB5") (pintype "bidirectional"))
     (pad "42" smd roundrect (at 0.25 -4.1625 90) (size 0.3 1.475) (layers "F.Cu" "F.Paste" "F.Mask") (roundrect_rratio 0.25)
-      (net 11 "/PTT1-IN") (pinfunction "PB6") (pintype "bidirectional"))
+      (net 60 "/IN1") (pinfunction "PB6") (pintype "bidirectional"))
     (pad "43" smd roundrect (at -0.25 -4.1625 90) (size 0.3 1.475) (layers "F.Cu" "F.Paste" "F.Mask") (roundrect_rratio 0.25)
-      (net 60 "/PTT2-IN") (pinfunction "PB7") (pintype "bidirectional"))
+      (net 40 "/IN2") (pinfunction "PB7") (pintype "bidirectional"))
     (pad "44" smd roundrect (at -0.75 -4.1625 90) (size 0.3 1.475) (layers "F.Cu" "F.Paste" "F.Mask") (roundrect_rratio 0.25)
       (net 50 "/BOOT0") (pinfunction "BOOT0") (pintype "input"))
@@
     (fp_line (start -0.8 0.4125) (end -0.8 -0.4125) (layer "F.Fab") (width 0.1))
     (pad "1" smd roundrect (at -0.825 0 270) (size 0.8 0.95) (layers "F.Cu" "F.Paste" "F.Mask") (roundrect_rratio 0.25)
-      (net 40 "/PTT2") (pintype "passive"))
+      (net 11 "/OUT2") (pintype "passive"))
     (pad "2" smd roundrect (at 0.825 0 270) (size 0.8 0.95) (layers "F.Cu" "F.Paste" "F.Mask") (roundrect_rratio 0.25)
       (net 54 "Net-(Q1-Pad2)") (pintype "passive"))
@@
   (segment (start 105.75 103.5) (end 106.2875 103.5) (width 0.25) (layer "B.Cu") (net 10))
   (segment (start 105.5 103.25) (end 105.75 103.5) (width 0.25) (layer "B.Cu") (net 10))
-  (segment (start 117.175 103.25) (end 116.75 103.25) (width 0.25) (layer "F.Cu") (net 11))
-  (segment (start 110.316891 99.624031) (end 109.69286 99) (width 0.25) (layer "F.Cu") (net 11))
-  (segment (start 116.75 103.25) (end 113.425816 99.925816) (width 0.25) (layer "F.Cu") (net 11))
-  (segment (start 109.69286 99) (end 108.5875 99) (width 0.25) (layer "F.Cu") (net 11))
-  (segment (start 113.425816 99.925816) (end 110.618676 99.925816) (width 0.25) (layer "F.Cu") (net 11))
-  (segment (start 110.618676 99.925816) (end 110.22143 99.52857) (width 0.25) (layer "F.Cu") (net 11))
+  (segment (start 115 105.072206) (end 115 106.175) (width 0.25) (layer "F.Cu") (net 11))
+  (segment (start 114.5 104.572206) (end 115 105.072206) (width 0.25) (layer "F.Cu") (net 11))
+  (segment (start 114.5 103.4125) (end 114.5 104.572206) (width 0.25) (layer "F.Cu") (net 11))
   (segment (start 109.05 96.0375) (end 108.5875 96.5) (width 0.25) (layer "F.Cu") (net 12))
   (segment (start 110.6 92.866006) (end 109.743948 92.866006) (width 0.25) (layer "F.Cu") (net 12))
@@
   (segment (start 116.5 105.75) (end 116.5 106.175) (width 0.25) (layer "F.Cu") (net 39))
   (segment (start 115 104.25) (end 116.5 105.75) (width 0.25) (layer "F.Cu") (net 39))
-  (segment (start 115 105.072206) (end 115 106.175) (width 0.25) (layer "F.Cu") (net 40))
-  (segment (start 114.5 104.572206) (end 115 105.072206) (width 0.25) (layer "F.Cu") (net 40))
-  (segment (start 114.5 103.4125) (end 114.5 104.572206) (width 0.25) (layer "F.Cu") (net 40))
+  (segment (start 110.432631 100.375489) (end 109.557142 99.5) (width 0.25) (layer "F.Cu") (net 40))
+  (segment (start 114.75 102.078928) (end 113.046561 100.375489) (width 0.25) (layer "F.Cu") (net 40))
+  (segment (start 116.75 104.75) (end 117.175 104.75) (width 0.25) (layer "F.Cu") (net 40))
+  (segment (start 116.168768 104.168768) (end 116.75 104.75) (width 0.25) (layer "F.Cu") (net 40))
+  (segment (start 114.75 102.15) (end 114.75 102.078928) (width 0.25) (layer "F.Cu") (net 40))
+  (segment (start 113.046561 100.375489) (end 110.432631 100.375489) (width 0.25) (layer "F.Cu") (net 40))
+  (segment (start 109.557142 99.5) (end 108.5875 99.5) (width 0.25) (layer "F.Cu") (net 40))
+  (segment (start 116.168768 103.551946) (end 116.168768 104.168768) (width 0.25) (layer "F.Cu") (net 40))
+  (via (at 116.168768 103.551946) (size 0.6) (drill 0.3) (layers "F.Cu" "B.Cu") (free) (net 40))
+  (via (at 114.75 102.15) (size 0.6) (drill 0.3) (layers "F.Cu" "B.Cu") (free) (net 40))
+  (segment (start 116.168768 103.551946) (end 116.151946 103.551946) (width 0.25) (layer "B.Cu") (net 40))
+  (segment (start 116.151946 103.551946) (end 114.75 102.15) (width 0.25) (layer "B.Cu") (net 40))
   (segment (start 118.75 97.75) (end 118.75 97.05) (width 0.3) (layer "F.Cu") (net 41))
   (segment (start 119 92) (end 119.525 92) (width 0.25) (layer "F.Cu") (net 41))
@@
   (segment (start 119.37452 102.37452) (end 119.75 102.75) (width 0.25) (layer "F.Cu") (net 59))
   (segment (start 119.75 102.75) (end 120.925 102.75) (width 0.25) (layer "F.Cu") (net 59))
-  (segment (start 110.432631 100.375489) (end 109.557142 99.5) (width 0.25) (layer "F.Cu") (net 60))
-  (segment (start 114.75 102.078928) (end 113.046561 100.375489) (width 0.25) (layer "F.Cu") (net 60))
-  (segment (start 116.75 104.75) (end 117.175 104.75) (width 0.25) (layer "F.Cu") (net 60))
-  (segment (start 116.168768 104.168768) (end 116.75 104.75) (width 0.25) (layer "F.Cu") (net 60))
-  (segment (start 114.75 102.15) (end 114.75 102.078928) (width 0.25) (layer "F.Cu") (net 60))
-  (segment (start 113.046561 100.375489) (end 110.432631 100.375489) (width 0.25) (layer "F.Cu") (net 60))
-  (segment (start 109.557142 99.5) (end 108.5875 99.5) (width 0.25) (layer "F.Cu") (net 60))
-  (segment (start 116.168768 103.551946) (end 116.168768 104.168768) (width 0.25) (layer "F.Cu") (net 60))
-  (via (at 116.168768 103.551946) (size 0.6) (drill 0.3) (layers "F.Cu" "B.Cu") (free) (net 60))
-  (via (at 114.75 102.15) (size 0.6) (drill 0.3) (layers "F.Cu" "B.Cu") (free) (net 60))
-  (segment (start 116.168768 103.551946) (end 116.151946 103.551946) (width 0.25) (layer "B.Cu") (net 60))
-  (segment (start 116.151946 103.551946) (end 114.75 102.15) (width 0.25) (layer "B.Cu") (net 60))
+  (segment (start 117.175 103.25) (end 116.75 103.25) (width 0.25) (layer "F.Cu") (net 60))
+  (segment (start 110.316891 99.624031) (end 109.69286 99) (width 0.25) (layer "F.Cu") (net 60))
+  (segment (start 116.75 103.25) (end 113.425816 99.925816) (width 0.25) (layer "F.Cu") (net 60))
+  (segment (start 109.69286 99) (end 108.5875 99) (width 0.25) (layer "F.Cu") (net 60))
+  (segment (start 113.425816 99.925816) (end 110.618676 99.925816) (width 0.25) (layer "F.Cu") (net 60))
+  (segment (start 110.618676 99.925816) (end 110.22143 99.52857) (width 0.25) (layer "F.Cu") (net 60))
   (segment (start 118.825 103.25) (end 118.25 103.25) (width 0.25) (layer "F.Cu") (net 61))
   (segment (start 118 103.5) (end 118 104) (width 0.25) (layer "F.Cu") (net 61))

Commit message: Added capability to use OPAMP1 for additional input gain and OPAMP2 to supply DC bias using the internal offset calibration feature
Parts:
- removed R3: 5.1K, Resistor_SMD:R_0603_1608Metric
- C11: value 10n/NP0 -> 4.7n/NP0
- R10, R11: value 2.2K -> 1.5K
- R14, R5: value 2.2K -> 5.1K
- moved C11 1.50 mm to (118.8, 93.5)
- moved R16 1.50 mm to (118.8, 95.0), turned to 180 degrees
- moved R5 1.50 mm to (118.8, 92.0), turned to 180 degrees
Connections:
- R16 pad 1: +3.3VA -> /ADC_BIAS
- R5 pad 1: /AFIN -> Net-(C14-Pad1)
- R5 pad 2: Net-(C14-Pad1) -> /AFIN
- U2 pad 15: unconnected-(U2-Pad15) -> /AFIN
- U2 pad 16: unconnected-(U2-Pad16) -> /ADC_BIAS
Routing:
- net /ADC_BIAS: track 0.00 -> 10.8 mm
- net /AFIN: track 11.1 -> 15.3 mm, vias 0 -> 2
- net +3.3VA: track 37.0 -> 35.3 mm
- net Net-(C14-Pad1): track 2.48 -> 1.40 mm
- net /RADIO-TX: track 27.4 -> 26.7 mm
- net +3V3: track 54.9 -> 54.3 mm
- net GND: vias 57 -> 56

Commit message: Modified DAC output to be able to handle line and mic level
Parts:
- R15, R17, R8, R9: value 220R -> 100R
- R18, R19, R4: value 220R -> 1.5K
- R2: value 10K -> 4.7K
- moved C12 1.06 mm to (122.5, 102.0), turned to 0 degrees
- moved R4 1.06 mm to (122.5, 100.5), turned to 0 degrees
Connections:
- C12 pad 1: Net-(C12-Pad1) -> /DAC_ATTEN
- C12 pad 2: GND -> Net-(C13-Pad1)
- C13 pad 1: Net-(C12-Pad1) -> Net-(C13-Pad1)
- R17 pad 1: Net-(C12-Pad1) -> Net-(C13-Pad1)
- R2 pad 1: Net-(C12-Pad1) -> Net-(C13-Pad1)
- R4 pad 2: Net-(C12-Pad1) -> Net-(C13-Pad1)
Routing:
- net Net-(C13-Pad1): track 0.00 -> 9.71 mm
- net Net-(C12-Pad1): track 9.64 -> 0.00 mm
- net GND: track 11.5 -> 10.2 mm, vias 56 -> 57
- net /DAC_ATTEN: track 5.38 -> 6.65 mm

Commit message: Bumped hardware version to 1.2 and generated fabrication data
Other:
- board text added: "AIOC V1.2"
- board text removed: "AIOC V1.1"
Changed lines of the file:
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@@
   (net 27 "/VIN")
   (net 28 "/VBUS")
-  (net 29 "Net-(C13-Pad1)")
+  (net 29 "Net-(C12-Pad2)")
   (net 30 "Net-(C14-Pad1)")
   (net 31 "Net-(J1-PadB5)")
@@
     (fp_line (start -0.8 -0.4125) (end 0.8 -0.4125) (layer "F.Fab") (width 0.1))
     (pad "1" smd roundrect (at -0.825 0 90) (size 0.8 0.95) (layers "F.Cu" "F.Paste" "F.Mask") (roundrect_rratio 0.25)
-      (net 29 "Net-(C13-Pad1)") (pintype "passive"))
+      (net 29 "Net-(C12-Pad2)") (pintype "passive"))
     (pad "2" smd roundrect (at 0.825 0 90) (size 0.8 0.95) (layers "F.Cu" "F.Paste" "F.Mask") (roundrect_rratio 0.25)
       (net 42 "/AFOUT") (pintype "passive"))
@@
       (net 57 "/DAC_ATTEN") (pintype "passive"))
     (pad "2" smd roundrect (at 0.775 0) (size 0.9 0.95) (layers "F.Cu" "F.Paste" "F.Mask") (roundrect_rratio 0.25)
-      (net 29 "Net-(C13-Pad1)") (pintype "passive"))
+      (net 29 "Net-(C12-Pad2)") (pintype "passive"))
     (model "${KICAD6_3DMODEL_DIR}/Capacitor_SMD.3dshapes/C_0603_1608Metric.wrl"
       (offset (xyz 0 0 0))
@@
       (net 1 "GND") (pintype "passive"))
     (pad "2" smd roundrect (at 0.825 0) (size 0.8 0.95) (layers "F.Cu" "F.Paste" "F.Mask") (roundrect_rratio 0.25)
-      (net 29 "Net-(C13-Pad1)") (pintype "passive"))
+      (net 29 "Net-(C12-Pad2)") (pintype "passive"))
     (model "${KICAD6_3DMODEL_DIR}/Resistor_SMD.3dshapes/R_0603_1608Metric.wrl"
       (offset (xyz 0 0 0))
@@
     (fp_line (start -0.8 0.4125) (end -0.8 -0.4125) (layer "F.Fab") (width 0.1))
     (pad "1" smd roundrect (at -0.825 0 180) (size 0.8 0.95) (layers "F.Cu" "F.Paste" "F.Mask") (roundrect_rratio 0.25)
-      (net 29 "Net-(C13-Pad1)") (pintype "passive"))
+      (net 29 "Net-(C12-Pad2)") (pintype "passive"))
     (pad "2" smd roundrect (at 0.825 0 180) (size 0.8 0.95) (layers "F.Cu" "F.Paste" "F.Mask") (roundrect_rratio 0.25)
       (net 57 "/DAC_ATTEN") (pintype "passive"))
@@
     (fp_line (start -0.8 -0.4) (end 0.8 -0.4) (layer "F.Fab") (width 0.1))
     (pad "1" smd roundrect (at -0.775 0 270) (size 0.9 0.95) (layers "F.Cu" "F.Paste" "F.Mask") (roundrect_rratio 0.25)
-      (net 29 "Net-(C13-Pad1)") (pintype "passive"))
+      (net 29 "Net-(C12-Pad2)") (pintype "passive"))
     (pad "2" smd roundrect (at 0.775 0 270) (size 0.9 0.95) (layers "F.Cu" "F.Paste" "F.Mask") (roundrect_rratio 0.25)
       (net 40 "/RADIO-MIC") (pintype "passive"))
@@
     (effects (font (size 0.4 0.4) (thickness 0.1)) (justify mirror))
   )
-  (gr_text "AIOC V1.1" (at 111.5 81.25) (layer "B.SilkS")
+  (gr_text "AIOC V1.2" (at 111.5 81.25) (layer "B.SilkS")
     (effects (font (size 1 1) (thickness 0.2)) (justify mirror))
   )

Commit message: Added an RC-lowpass to ADC BIAS net just to be safe
Parts:
- added C16: 100n, Capacitor_SMD:C_0603_1608Metric, F.Cu at (118.8, 93.5)
- added R3: 100R, Resistor_SMD:R_0603_1608Metric, F.Cu at (118.8, 97.2)
- moved C11 3.00 mm to (118.8, 90.5)
Connections:
- R16 pad 1: /ADC_BIAS -> Net-(R16-Pad1)
Routing:
- net /ADC_BIAS: track 10.8 -> 6.43 mm
- net Net-(R16-Pad1): track 0.00 -> 3.60 mm
- net /RADIO-TX: track 26.7 -> 23.9 mm
- net /AFIN: track 15.5 -> 16.3 mm
- net GND: vias 57 -> 56

Commit message: Switched to a different USB-C socket, which is more easily sourced from alternative sources
Parts:
- J1: value 12401832E402A -> USB4105-GF-A; footprint AIOC:USB_C_Receptacle_Amphenol_12401832E40-2A -> AIOC:USB_C_Receptacle_GCT_USB4105-xx-A_16P_TopMnt_Horizontal
- moved J1 1.45 mm to (111.5, 83.5)
Connections:
- net Net-(J1-PadA5) renamed /CC1
- net Net-(J1-PadB5) renamed /CC2
Routing:
- net /SWO: track 18.1 -> 22.2 mm
- net /CC2: track 8.97 -> 11.8 mm
- net /SWDIO: track 15.4 -> 17.8 mm
- net /USB-DN: track 14.0 -> 12.2 mm, vias 3 -> 2
- net GND: track 10.2 -> 9.29 mm, vias 56 -> 52
- net /SWCLK: track 20.0 -> 20.6 mm
- net /CC1: track 10.1 -> 10.5 mm, vias 2 -> 0
- net /USB-DP: vias 3 -> 2
Other:
- board text removed: "BOOT"
