File: kicad/k1-aioc/k1-aioc.kicad_sch (KiCad schematic)
At the start: 48 parts, among them J1 12401832E402A, J2 Conn_01x07_Male, Q1 BC847BS, U1 MIC5330-SSYML, U2 STM32F373CBTx, Y1 8MHz/20pF

Commit message: Changed naming of microcontroller IO pins to IN/OUT
Connections:
- net PTT1 renamed OUT1
- net PTT1-IN renamed IN1
- net PTT2 renamed OUT2
- net PTT2-IN renamed IN2
Changed lines of the file:
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@@
     (effects (font (size 1.27 1.27)) (justify left bottom))
   )
-  (label "PTT2-IN" (at 142.24 154.94 0)
+  (label "IN2" (at 142.24 154.94 0)
     (effects (font (size 1.27 1.27)) (justify left bottom))
   )
@@
     (effects (font (size 1.27 1.27)) (justify left bottom))
   )
-  (label "PTT1-IN" (at 142.24 152.4 0)
+  (label "IN1" (at 142.24 152.4 0)
     (effects (font (size 1.27 1.27)) (justify left bottom))
   )
@@
     (effects (font (size 1.27 1.27)) (justify left bottom))
   )
-  (label "PTT2" (at 142.24 96.52 0)
+  (label "OUT2" (at 142.24 96.52 0)
     (effects (font (size 1.27 1.27)) (justify left bottom))
   )
@@
     (effects (font (size 1.27 1.27)) (justify left bottom))
   )
-  (label "PTT1" (at 142.24 99.06 0)
+  (label "OUT1" (at 142.24 99.06 0)
     (effects (font (size 1.27 1.27)) (justify left bottom))
   )

Commit message: Added capability to use OPAMP1 for additional input gain and OPAMP2 to supply DC bias using the internal offset calibration feature
Parts:
- removed R5: 2.2K, Resistor_SMD:R_0603_1608Metric, symbol Device:R
- C11: value 10n/NP0 -> 4.7n/NP0; LCSC C57112 -> C53987
- R10, R11: value 2.2K -> 1.5K; LCSC C4190 -> C22843
- R14: value 2.2K -> 5.1K; LCSC C4190 -> C23186
- renumbered R3 to R5
Connections:
- net +3.3VA: no longer R16.1
- net AFIN: now also U2.15 (PA5)
- net GND: no longer R5.1
- net at C14.1: now also R5.1
- net ADC_BIAS: now reaches U2.16 (PA6)
- net ADC_BIAS: now also R16.1
Other:
- note added: "OPAMP1_VINP"
- note added: "OPAMP2_VOUT"
- note added: "PB2 is used when Gain=1 (Input range 0-6.6V) for legacy reasons (V1.0 hardware) For gains x2/x4/x8/x16, OPAMP1 is used. Correct scaled-down ADC bias is supplied via OPAMP2"
- moved on the sheet: R16, R5

Commit message: Modified DAC output to be able to handle line and mic level
Parts:
- R15, R8, R9: value 220R -> 100R; LCSC C22962 -> C22775
- R17: value 220R -> 100R; LCSC (none) -> C22775
- R18, R19, R4: value 220R -> 1.5K; LCSC C22962 -> C22843
- R2: value 10K -> 4.7K; LCSC C25804 -> C23162
Connections:
- net DAC_ATTEN: now also C12.1
- net GND: no longer C12.2
- net at C13.1, R17.1, R2.1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: now also C12.2; no longer C12.1
Other:
- note added: "For legacy reasons (V1.0 hardware) PB2 is used when Gain=1 (Input range 0-6.6V) and bias is supplied with static voltage divider For gains x2/x4/x8/x16, OPAMP1 is used. Correct scaled-down ADC bias is supplied via OPAMP2"
- note added: "Maximum DAC Load 5Kohm Output Level 350mVpk @ 10Kohm load Output impedance approx. 1.3Kohm With Attenuator: Output Level 35mVpk Output impedance approx. 90Ohm"
- note removed: "PB2 is used when Gain=1 (Input range 0-6.6V) for legacy reasons (V1.0 hardware) For gains x2/x4/x8/x16, OPAMP1 is used. Correct scaled-down ADC bias is supplied via OPAMP2"
- moved on the sheet: C12, R10, R11, R17, R2, R8, R9

Commit message: Added an RC-lowpass to ADC BIAS net just to be safe
Parts:
- added C16: 100n, Capacitor_SMD:C_0603_1608Metric, symbol Device:C
- added R3: 100R, Resistor_SMD:R_0603_1608Metric, symbol Device:R
Connections:
- net ADC_BIAS: now also R3.2; no longer R16.1
- net GND: now also C16.1
- new net: C16.2, R16.1, R3.1
Other:
- moved on the sheet: R16
Changed lines of the file:
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@@
   (junction (at 143.51 33.02) (diameter 0) (color 0 0 0 0)
   )
+  (junction (at 200.66 111.76) (diameter 0) (color 0 0 0 0)
+  )
   (junction (at 93.98 35.56) (diameter 0) (color 0 0 0 0)
   )
@@
   )
   (wire (pts (xy 170.18 176.53) (xy 171.45 176.53))
+    (stroke (width 0) (type default) (color 0 0 0 0))
+  )
+  (wire (pts (xy 212.09 111.76) (xy 200.66 111.76))
     (stroke (width 0) (type default) (color 0 0 0 0))
   )
@@
     (stroke (width 0) (type default) (color 0 0 0 0))
   )
-  (wire (pts (xy 139.7 111.76) (xy 200.66 111.76))
+  (wire (pts (xy 139.7 111.76) (xy 186.69 111.76))
     (stroke (width 0) (type default) (color 0 0 0 0))
   )
@@
     (stroke (width 0) (type default) (color 0 0 0 0))
   )
+  (wire (pts (xy 194.31 111.76) (xy 200.66 111.76))
+    (stroke (width 0) (type default) (color 0 0 0 0))
+  )
   (wire (pts (xy 194.31 104.14) (xy 200.66 104.14))
     (stroke (width 0) (type default) (color 0 0 0 0))
@@
     (stroke (width 0) (type default) (color 0 0 0 0))
   )
-  (wire (pts (xy 200.66 111.76) (xy 200.66 132.08))
+  (wire (pts (xy 200.66 111.76) (xy 200.66 125.73))
     (stroke (width 0) (type default) (color 0 0 0 0))
   )
@@
     (stroke (width 0) (type default) (color 0 0 0 0))
   )
-  (wire (pts (xy 200.66 139.7) (xy 200.66 142.24))
+  (wire (pts (xy 212.09 133.35) (xy 212.09 135.89))
+    (stroke (width 0) (type default) (color 0 0 0 0))
+  )
+  (wire (pts (xy 200.66 133.35) (xy 200.66 142.24))
     (stroke (width 0) (type default) (color 0 0 0 0))
   )
@@
   )
   (wire (pts (xy 152.4 157.48) (xy 152.4 162.56))
+    (stroke (width 0) (type default) (color 0 0 0 0))
+  )
+  (wire (pts (xy 212.09 125.73) (xy 212.09 111.76))
     (stroke (width 0) (type default) (color 0 0 0 0))
   )
@@
     (pin "2")
   )
+  (symbol (lib_id "Device:R") (at 190.5 111.76 270) (unit 1)
+    (in_bom yes) (on_board yes)
+    (property "Reference" "R3" (id 0) (at 190.5 114.3 90))
+    (property "Value" "100R" (id 1) (at 196.85 114.3 90))
+    (property "Footprint" "Resistor_SMD:R_0603_1608Metric" (id 2) (at 190.5 109.982 90)
+      (effects (font (size 1.27 1.27)) hide)
+    )
+    (property "Datasheet" "~" (id 3) (at 190.5 111.76 0)
+      (effects (font (size 1.27 1.27)) hide)
+    )
+    (property "LCSC" "C22775" (id 4) (at 190.5 114.3 0)
+      (effects (font (size 1.27 1.27)) hide)
+    )
+    (pin "1")
+    (pin "2")
+  )
   (symbol (lib_id "Device:R") (at 190.5 119.38 270) (unit 1)
     (in_bom yes) (on_board yes)
@@
     (pin "2")
   )
-  (symbol (lib_id "Device:R") (at 200.66 135.89 0) (unit 1)
-    (in_bom yes) (on_board yes) (fields_autoplaced)
-    (property "Reference" "R16" (id 0) (at 203.2 134.6199 0)
-      (effects (font (size 1.27 1.27)) (justify left))
-    )
-    (property "Value" "5.1K" (id 1) (at 203.2 137.1599 0)
-      (effects (font (size 1.27 1.27)) (justify left))
-    )
-    (property "Footprint" "Resistor_SMD:R_0603_1608Metric" (id 2) (at 198.882 135.89 90)
-      (effects (font (size 1.27 1.27)) hide)
-    )
-    (property "Datasheet" "~" (id 3) (at 200.66 135.89 0)
-      (effects (font (size 1.27 1.27)) hide)
-    )
-    (property "LCSC" "C23186" (id 4) (at 198.12 137.1601 0)
+  (symbol (lib_id "Device:R") (at 200.66 129.54 0) (unit 1)
+    (in_bom yes) (on_board yes) (fields_autoplaced)
+    (property "Reference" "R16" (id 0) (at 203.2 128.2699 0)
+      (effects (font (size 1.27 1.27)) (justify left))
+    )
+    (property "Value" "5.1K" (id 1) (at 203.2 130.8099 0)
+      (effects (font (size 1.27 1.27)) (justify left))
+    )
+    (property "Footprint" "Resistor_SMD:R_0603_1608Metric" (id 2) (at 198.882 129.54 90)
+      (effects (font (size 1.27 1.27)) hide)
+    )
+    (property "Datasheet" "~" (id 3) (at 200.66 129.54 0)
+      (effects (font (size 1.27 1.27)) hide)
+    )
+    (property "LCSC" "C23186" (id 4) (at 198.12 130.8101 0)
       (effects (font (size 1.27 1.27)) hide)
     )
@@
     (pin "S1")
   )
+  (symbol (lib_id "Device:C") (at 212.09 129.54 180) (unit 1)
+    (in_bom yes) (on_board yes) (fields_autoplaced)
+    (property "Reference" "C16" (id 0) (at 215.9 128.2699 0)
+      (effects (font (size 1.27 1.27)) (justify right))
+    )
+    (property "Value" "100n" (id 1) (at 215.9 130.8099 0)
+      (effects (font (size 1.27 1.27)) (justify right))
+    )
+    (property "Footprint" "Capacitor_SMD:C_0603_1608Metric" (id 2) (at 211.1248 125.73 0)
+      (effects (font (size 1.27 1.27)) hide)
+    )
+    (property "Datasheet" "~" (id 3) (at 212.09 129.54 0)
+      (effects (font (size 1.27 1.27)) hide)
+    )
+    (property "LCSC" "C14663" (id 4) (at 208.28 130.8101 0)
+      (effects (font (size 1.27 1.27)) hide)
+    )
+    (pin "1")
+    (pin "2")
+  )
   (symbol (lib_id "Device:R") (at 176.53 152.4 270) (unit 1)
     (in_bom yes) (on_board yes)
@@
     (pin "2")
   )
+  (symbol (lib_id "power:GND") (at 212.09 135.89 0) (unit 1)
+    (in_bom yes) (on_board yes) (fields_autoplaced)
+    (property "Reference" "#PWR0127" (id 0) (at 212.09 142.24 0)
+      (effects (font (size 1.27 1.27)) hide)
+    )
+    (property "Value" "GND" (id 1) (at 212.09 140.97 0))
+    (property "Footprint" "" (id 2) (at 212.09 135.89 0)
+      (effects (font (size 1.27 1.27)) hide)
+    )
+    (property "Datasheet" "" (id 3) (at 212.09 135.89 0)
+      (effects (font (size 1.27 1.27)) hide)
+    )
+    (pin "1")
+  )
   (symbol (lib_id "Connector:Conn_01x07_Male") (at 33.02 123.19 0) (mirror x) (unit 1)
     (in_bom yes) (on_board yes)
@@
       (reference "#PWR0126") (unit 1) (value "GND") (footprint "")
     )
+    (path "/ea68b534-7587-4b23-aa5b-b6cdceb80af1"
+      (reference "#PWR0127") (unit 1) (value "GND") (footprint "")
+    )
     (path "/4f4a10d7-b161-42d7-90b7-9b7948641a9a"
       (reference "C1") (unit 1) (value "22p/NP0") (footprint "Capacitor_SMD:C_0603_1608Metric")
@@
       (reference "C15") (unit 1) (value "100n") (footprint "Capacitor_SMD:C_0603_1608Metric")
     )
+    (path "/c6f4af78-42df-40f1-8a39-7b57940af9c3"
+      (reference "C16") (unit 1) (value "100n") (footprint "Capacitor_SMD:C_0603_1608Metric")
+    )
     (path "/44eaa438-6c06-4723-b7a3-c2f7fc0b787d"
       (reference "D1") (unit 1) (value "GREEN") (footprint "LED_SMD:LED_0603_1608Metric")
@@
       (reference "R2") (unit 1) (value "4.7K") (footprint "Resistor_SMD:R_0603_1608Metric")
     )
+    (path "/7a96bc4e-e7fc-4000-ada6-0e57b4b16bd9"
+      (reference "R3") (unit 1) (value "100R") (footprint "Resistor_SMD:R_0603_1608Metric")
+    )
     (path "/a9b02ec6-e6e2-4eac-8da5-3da941741fdc"

Commit message: Switched to a different USB-C socket, which is more easily sourced from alternative sources
Parts:
- J1: value 12401832E402A -> USB4105-GF-A; footprint AIOC:USB_C_Receptacle_Amphenol_12401832E40-2A -> AIOC:USB_C_Receptacle_GCT_USB4105-xx-A_16P_TopMnt_Horizontal; LCSC C464604 -> C2988369
Connections:
- net CC2: now reaches J1.B5 (CC2), R6.2
- net CC1: now reaches J1.A5 (CC1), R7.2
Changed lines of the file:
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@@
+    (effects (font (size 1.27 1.27)) (justify left bottom))
+  )
+  (label "CC2" (at 55.88 40.64 0)
     (effects (font (size 1.27 1.27)) (justify left bottom))
   )
@@
   )
   (label "RADIO-TX" (at 238.76 119.38 0)
+    (effects (font (size 1.27 1.27)) (justify left bottom))
+  )
+  (label "CC1" (at 55.88 38.1 0)
     (effects (font (size 1.27 1.27)) (justify left bottom))
   )
@@
     (in_bom yes) (on_board yes) (fields_autoplaced)
     (property "Reference" "J1" (id 0) (at 36.83 25.4 0))
-    (property "Value" "12401832E402A" (id 1) (at 36.83 27.94 0))
-    (property "Footprint" "AIOC:USB_C_Receptacle_Amphenol_12401832E40-2A" (id 2) (at 40.64 48.26 0)
+    (property "Value" "USB4105-GF-A" (id 1) (at 36.83 27.94 0))
+    (property "Footprint" "AIOC:USB_C_Receptacle_GCT_USB4105-xx-A_16P_TopMnt_Horizontal" (id 2) (at 40.64 48.26 0)
       (effects (font (size 1.27 1.27)) hide)
     )
@@
       (effects (font (size 1.27 1.27)) hide)
     )
-    (property "LCSC" "C464604" (id 4) (at 36.83 25.4 0)
+    (property "LCSC" "C2988369" (id 4) (at 36.83 25.4 0)
       (effects (font (size 1.27 1.27)) hide)
     )
@@
     )
     (path "/c5b80805-bc26-457d-a1fd-cf6a8b83ea3f"
-      (reference "J1") (unit 1) (value "12401832E402A") (footprint "AIOC:USB_C_Receptacle_Amphenol_12401832E40-2A")
+      (reference "J1") (unit 1) (value "USB4105-GF-A") (footprint "AIOC:USB_C_Receptacle_GCT_USB4105-xx-A_16P_TopMnt_Horizontal")
     )
     (path "/f2c9e50d-789f-4fc9-bf13-807bdf38a185"
